Commit message: Robot built with joints in correct positions. PIDs need better tuning, and joint limits need to be set. Basic control script added

File: inchworm_description/urdf/updated_description.urdf (robot description, URDF)
Before this commit: robot inchworm, 7 links, 6 joints
Joints:
- joint link1_to_foot: axis 0 0 1 -> 0 1 0
- joint link2_to_link1: origin xyz=0 0.1625 -0.001 rpy=3.14 3.14 -1.57 -> xyz=0 0 -0.001 rpy=0 0 0
- joint link3_to_link2: origin xyz=0.165 0 -0.001 rpy=3.14 0 0 -> xyz=0.165 0 -0.001 rpy=3.14 0 3.14
- joint link3_to_link4: origin xyz=0.055 0 0 rpy=0 0 0 -> xyz=-0.165 0 0 rpy=0 0 0
- joint link4_to_foot: origin xyz=0.051 0 0 rpy=0 1.57 0 -> xyz=0 0 0 rpy=0 -1.57 0

Commit message: Moveit package

File: inchworm_description/urdf/updated_description.urdf (robot description, URDF)
Before this commit: robot inchworm, 7 links, 6 joints
Joints:
- joint link2_to_link1: origin xyz=0 0 -0.001 rpy=0 0 0 -> xyz=0 0 -0.001 rpy=0 0 1.57

Commit message: Added and aligned collisions to updated_urdf

File: inchworm_description/urdf/updated_description.urdf (robot description, URDF)
Before this commit: robot inchworm, 7 links, 6 joints
Links:
- link foot: geometry collision box size=0.07 0.07 0.05463; visual mesh filename=package://inchworm_description/media/link0.stl scale=0.001 0.001 0.001
- link link1: geometry collision box size=0.045 0.08 0.08; visual mesh filename=package://inchworm_description/media/link1.stl scale=0.001 0.001 0.001
- link link2: geometry collision box size=0.22 0.05 0.08; visual mesh filename=package://inchworm_description/media/link2.stl scale=0.001 0.001 0.001
- link link3: geometry collision box size=0.22 0.05 0.08; visual mesh filename=package://inchworm_description/media/link3.stl scale=0.001 0.001 0.001
- link link4: geometry collision box size=0.08 0.045 0.08; visual mesh filename=package://inchworm_description/media/link4.stl scale=0.001 0.001 0.001
- link other_foot: geometry collision box size=0.07 0.07 0.05463; visual mesh filename=package://inchworm_description/media/link5.stl scale=0.001 0.001 0.001

Commit message: Moving frames slightly

File: inchworm_description/urdf/updated_description.urdf (robot description, URDF)
Before this commit: robot inchworm, 7 links, 6 joints
Joints:
- joint link4_to_foot: origin xyz=0 0 0 rpy=0 -1.57 0 -> xyz=-0.105 0 0 rpy=0 -1.57 0

Commit message: Move script working but not returning any valid IK solutions

File: inchworm_description/urdf/updated_description.urdf (robot description, URDF)
Before this commit: robot inchworm, 7 links, 6 joints
Joints:
- joint link1_to_foot: limit lower=0 upper=6.28 effort=10 velocity=1.0 -> lower=-6.28 upper=6.28 effort=10 velocity=1.0
- joint link2_to_link1: limit lower=0 upper=6.28 effort=10 velocity=1.0 -> lower=-6.28 upper=6.28 effort=10 velocity=1.0
- joint link3_to_link2: limit lower=0 upper=6.28 effort=10 velocity=1.0 -> lower=-6.28 upper=6.28 effort=10 velocity=1.0
- joint link3_to_link4: limit lower=0 upper=6.28 effort=10 velocity=1.0 -> lower=-6.28 upper=6.28 effort=10 velocity=1.0
- joint link4_to_foot: limit lower=0 upper=6.28 effort=10 velocity=1.0 -> lower=-6.28 upper=6.28 effort=10 velocity=1.0

Commit message: Reducing joint limits allows for trajectory planning!

File: inchworm_description/urdf/updated_description.urdf (robot description, URDF)
Before this commit: robot inchworm, 7 links, 6 joints
Joints:
- joint link1_to_foot: limit lower=-6.28 upper=6.28 effort=10 velocity=1.0 -> lower=-3.14 upper=3.14 effort=10 velocity=1.0
- joint link2_to_link1: limit lower=-6.28 upper=6.28 effort=10 velocity=1.0 -> lower=-3.14 upper=3.14 effort=10 velocity=1.0
- joint link3_to_link2: limit lower=-6.28 upper=6.28 effort=10 velocity=1.0 -> lower=-3.14 upper=3.14 effort=10 velocity=1.0
- joint link3_to_link4: limit lower=-6.28 upper=6.28 effort=10 velocity=1.0 -> lower=-3.14 upper=3.14 effort=10 velocity=1.0
- joint link4_to_foot: limit lower=-6.28 upper=6.28 effort=10 velocity=1.0 -> lower=-3.14 upper=3.14 effort=10 velocity=1.0

Commit message: Removed old sim files and added magnet sim

File: inchworm_description/urdf/updated_description.urdf (robot description, URDF)
Before this commit: robot inchworm, 7 links, 6 joints
Links:
- removed link foot
- removed link link1
- removed link link2
- added link iw_ankle_bottom, mass 0.151; collision box size=0.22 0.05 0.08; visual mesh filename=package://inchworm_description/media/link2.stl scale=0.001 0.001 0.001
- added link iw_foot_bottom, mass 0.151; collision box size=0.07 0.07 0.05463; visual mesh filename=package://inchworm_description/media/link0.stl scale=0.001 0.001 0.001
Joints:
- removed joint foot_to_world
- removed joint link1_to_foot
- removed joint link2_to_link1
- added joint iw_ankle_bottom_to_foot: type revolute, parent iw_foot_bottom, child link1, origin xyz=0 0 0.05463 rpy=1.57 0 0, axis 0 1 0, limit lower=-3.14 upper=3.14 effort=10 velocity=1.0
- added joint iw_ankle_bottom_to_link1: type revolute, parent link1, child iw_ankle_bottom, origin xyz=0 0 -0.001 rpy=0 0 1.57, axis 0 0 1, limit lower=-3.14 upper=3.14 effort=10 velocity=1.0
- added joint iw_foot_bottom_to_world: type fixed, parent world, child iw_foot_bottom, origin xyz=0 0 0.05537 rpy=0 0 0
- joint link3_to_link2: parent link2 -> iw_ankle_bottom

Commit message: Negate the second joint direction so that all joint angles are positive

File: inchworm_description/urdf/updated_description.urdf (robot description, URDF)
Before this commit: robot inchworm, 7 links, 6 joints
Joints:
- joint link2_to_link1: axis 0 0 1 -> 0 0 -1

Commit message: Updated link and joint naming conventions

File: inchworm_description/urdf/updated_description.urdf (robot description, URDF)
Before this commit: robot inchworm, 7 links, 6 joints
Links:
- removed link foot
- removed link link1
- removed link link2
- removed link link3
- removed link link4
- removed link other_foot
- added link iw_ankle_bottom, mass 0.151; collision box size=0.045 0.08 0.08; visual mesh filename=package://inchworm_description/media/link1.stl scale=0.001 0.001 0.001
- added link iw_ankle_top, mass 0.151; collision box size=0.08 0.045 0.08; visual mesh filename=package://inchworm_description/media/link4.stl scale=0.001 0.001 0.001
- added link iw_beam_bottom, mass 0.151; collision box size=0.22 0.05 0.08; visual mesh filename=package://inchworm_description/media/link2.stl scale=0.001 0.001 0.001
- added link iw_beam_top, mass 0.151; collision box size=0.22 0.05 0.08; visual mesh filename=package://inchworm_description/media/link3.stl scale=0.001 0.001 0.001
- added link iw_foot_bottom, mass 0.151; collision box size=0.07 0.07 0.05463; visual mesh filename=package://inchworm_description/media/link0.stl scale=0.001 0.001 0.001
- added link iw_foot_top, mass 0.151; collision box size=0.07 0.07 0.05463; visual mesh filename=package://inchworm_description/media/link5.stl scale=0.001 0.001 0.001
Joints:
- removed joint link1_to_foot
- removed joint link2_to_link1
- removed joint link3_to_link2
- removed joint link3_to_link4
- removed joint link4_to_foot
- added joint iw_ankle_foot_bottom: type revolute, parent iw_foot_bottom, child iw_ankle_bottom, origin xyz=0 0 0.05463 rpy=1.57 0 0, axis 0 1 0, limit lower=-3.14 upper=3.14 effort=10 velocity=1.0
- added joint iw_ankle_foot_top: type revolute, parent iw_ankle_top, child iw_foot_top, origin xyz=-0.105 0 0 rpy=0 -1.57 0, axis 0 0 1, limit lower=-3.14 upper=3.14 effort=10 velocity=1.0
- added joint iw_beam_ankle_bottom: type revolute, parent iw_ankle_bottom, child iw_beam_bottom, origin xyz=0 0 -0.001 rpy=0 0 1.57, axis 0 0 -1, limit lower=-3.14 upper=3.14 effort=10 velocity=1.0
- added joint iw_beam_ankle_top: type revolute, parent iw_beam_top, child iw_ankle_top, origin xyz=-0.165 0 0 rpy=0 0 0, axis 0 0 1, limit lower=-3.14 upper=3.14 effort=10 velocity=1.0
- added joint iw_mid_joint: type revolute, parent iw_beam_bottom, child iw_beam_top, origin xyz=0.165 0 -0.001 rpy=3.14 0 3.14, axis 0 0 1, limit lower=-3.14 upper=3.14 effort=10 velocity=1.0
- joint foot_to_world: child foot -> iw_foot_bottom

Commit message: Flip direction of end effector joints

File: inchworm_description/urdf/updated_description.urdf (robot description, URDF)
Before this commit: robot inchworm, 7 links, 6 joints
Joints:
- joint iw_ankle_foot_bottom: axis 0 1 0 -> 0 -1 0
- joint iw_ankle_foot_top: axis 0 0 1 -> 0 0 -1

Commit message: Robot model with new STLs functional

File: inchworm_description/urdf/updated_description.urdf (robot description, URDF)
Before this commit: robot inchworm, 7 links, 6 joints
Links:
- link iw_ankle_bottom: geometry collision box size=0.045 0.08 0.08; visual mesh filename=package://inchworm_description/media/ankle.stl scale=0.001 0.001 0.001
- link iw_beam_bottom: geometry collision box size=0.22 0.05 0.08; visual mesh filename=package://inchworm_description/media/beam_bottom.stl scale=0.001 0.001 0.001
- link iw_foot_bottom: geometry collision box size=0.07 0.07 0.05463; visual mesh filename=package://inchworm_description/media/ee.stl scale=0.001 0.001 0.001
- link iw_foot_top: geometry collision box size=0.07 0.07 0.05463; visual mesh filename=package://inchworm_description/media/ee.stl scale=0.001 0.001 0.001
Joints:
- joint iw_ankle_foot_bottom: origin xyz=0 0 0.05463 rpy=1.57 0 0 -> xyz=0 0 0.0625 rpy=1.57 0 0
- joint iw_ankle_foot_top: origin xyz=-0.105 0 0 rpy=0 -1.57 0 -> xyz=-0.0625 0 0 rpy=0 1.57 0
- joint iw_beam_ankle_bottom: origin xyz=0 0 -0.001 rpy=0 0 1.57 -> xyz=0 0 0.001 rpy=0 0 1.57
