Commit message: Update sdf generation

File: inchworm_description/urdf/shingle_description.urdf (robot description, URDF)
Before this commit: robot shingle, 2 links, 0 joints
Links:
- removed link world

Commit message: Inchworm and shingle loading in, on top of each other

File: inchworm_description/urdf/shingle_description.urdf (robot description, URDF)
Before this commit: robot shingle, 1 links, 0 joints
Links:
- link shingle: geometry collision box size=0.254 0.182 0.02; visual box size=0.254 0.182 0.02

Commit message: Inchworm and shingle visualize in gazebo and rviz, and move with each other

File: inchworm_description/urdf/shingle_description.urdf (robot description, URDF)
Before this commit: robot shingle, 1 links, 0 joints
Links:
- removed link shingle
- added link shingle/shingle, mass 0.151; collision box size=0.254 0.182 0.02; visual box size=0.254 0.182 0.02

Commit message: Its doing magnety things, kind of

File: inchworm_description/urdf/shingle_description.urdf (robot description, URDF)
Before this commit: robot shingle, 1 links, 0 joints
Links:
- link shingle/shingle: geometry visual box size=0.254 0.182 0.02
