Commit message: Outdated STLs loading in right place with joints

File: inchworm_description/urdf/inchworm_description.urdf (robot description, URDF)
Before this commit: robot inchworm, 5 links, 4 joints
Links:
- link link_1: geometry collision mesh filename=package://inchworm_description/media/link1.stl scale=0.001 0.001 0.001; visual mesh filename=package://inchworm_description/media/link1.stl scale=0.001 0.001 0.001
- link link_2: geometry collision mesh filename=package://inchworm_description/media/link2.stl scale=0.001 0.001 0.001; visual mesh filename=package://inchworm_description/media/link2.stl scale=0.001 0.001 0.001
- link link_3: geometry collision mesh filename=package://inchworm_description/media/link3.stl scale=0.001 0.001 0.001; visual mesh filename=package://inchworm_description/media/link3.stl scale=0.001 0.001 0.001
- link link_4: geometry collision mesh filename=package://inchworm_description/meshes/link4.stl scale=0.001 0.001 0.001; visual mesh filename=package://inchworm_description/meshes/link4.stl scale=0.001 0.001 0.001

Commit message: Refactor mesh files and urdf naming

File: inchworm_description/urdf/inchworm_description.urdf (robot description, URDF)
Before this commit: robot inchworm, 7 links, 6 joints
Links:
- link iw_ankle_bottom: geometry collision box size=0.045 0.08 0.08; visual mesh filename=package://inchworm_description/meshes/ankle.stl scale=0.001 0.001 0.001
- link iw_ankle_top: geometry collision box size=0.08 0.045 0.08; visual mesh filename=package://inchworm_description/meshes/ankle.stl scale=0.001 0.001 0.001
- link iw_beam_bottom: geometry collision box size=0.22 0.05 0.08; visual mesh filename=package://inchworm_description/meshes/beam_bottom.stl scale=0.001 0.001 0.001
- link iw_beam_top: geometry collision box size=0.22 0.05 0.08; visual mesh filename=package://inchworm_description/meshes/beam_top.stl scale=0.001 0.001 0.001
- link iw_foot_bottom: geometry collision box size=0.07 0.07 0.05463; visual mesh filename=package://inchworm_description/meshes/ee.stl scale=0.001 0.001 0.001
- link iw_foot_top: geometry collision box size=0.07 0.07 0.05463; visual mesh filename=package://inchworm_description/meshes/ee.stl scale=0.001 0.001 0.001

Commit message: updated_description->inchworm_description. MoveIt now connected properly and working with new model.

File: inchworm_description/urdf/inchworm_description.urdf (robot description, URDF)
Before this commit: robot inchworm, 7 links, 6 joints
Joints:
- joint foot_to_world: origin xyz=0 0 0.05537 rpy=0 0 0 -> xyz=0 0 0 rpy=0 0 0
- joint iw_ankle_foot_bottom: origin xyz=0 0 0.0625 rpy=1.57 0 0 -> xyz=0 0 0.105 rpy=1.57 0 0
- joint iw_ankle_foot_top: origin xyz=-0.0625 0 0 rpy=0 1.57 0 -> xyz=-0.105 0 0 rpy=0 1.57 0
- joint iw_beam_ankle_bottom: limit lower=-3.14 upper=3.14 effort=10 velocity=1.0 -> lower=-0.785 upper=3.14 effort=10 velocity=1.0
- joint iw_beam_ankle_top: limit lower=-3.14 upper=3.14 effort=10 velocity=1.0 -> lower=-0.785 upper=3.14 effort=10 velocity=1.0
- joint iw_mid_joint: limit lower=-3.14 upper=3.14 effort=10 velocity=1.0 -> lower=-0.785 upper=3.14 effort=10 velocity=1.0

Commit message: Finally getting gazebo to behave again.

File: inchworm_description/urdf/inchworm_description.urdf (robot description, URDF)
Before this commit: robot inchworm, 7 links, 6 joints
Links:
- removed link world
- added link iw_root
Joints:
- removed joint foot_to_world
- added joint foot_to_root: type fixed, parent iw_root, child iw_foot_bottom, origin xyz=0 0 0 rpy=0 0 0, limit lower=0 upper=0 effort=10 velocity=10

Commit message: Part way through updating STLs

File: inchworm_description/urdf/inchworm_description.urdf (robot description, URDF)
Before this commit: robot inchworm, 7 links, 6 joints
Links:
- link iw_ankle_bottom: geometry collision box size=0.045 0.08 0.08; visual mesh filename=package://inchworm_description/meshes/ankle_bottom.stl scale=0.001 0.001 0.001

Commit message: First ankle needs to be rotated 180 about z axis, might fix offsets

File: inchworm_description/urdf/inchworm_description.urdf (robot description, URDF)
Before this commit: robot inchworm, 7 links, 6 joints
Links:
- link iw_ankle_top: geometry collision box size=0.08 0.045 0.08; visual mesh filename=package://inchworm_description/meshes/ankle_top.stl scale=0.001 0.001 0.001
Joints:
- joint iw_ankle_foot_bottom: origin xyz=0 0 0.105 rpy=1.57 0 0 -> xyz=0 0.0075 0.109 rpy=1.57 0 0
- joint iw_ankle_foot_top: origin xyz=-0.105 0 0 rpy=0 1.57 0 -> xyz=-0.109 0 0 rpy=0 1.57 0

Commit message: New robot model

File: inchworm_description/urdf/inchworm_description.urdf (robot description, URDF)
Before this commit: robot inchworm, 7 links, 6 joints
Joints:
- joint iw_ankle_foot_top: origin xyz=-0.109 0 0 rpy=0 1.57 0 -> xyz=-0.109 0 -0.008 rpy=0 1.57 0
- joint iw_beam_ankle_bottom: origin xyz=0 0 0.001 rpy=0 0 1.57 -> xyz=0 0 0.0165 rpy=0 0 1.57
- joint iw_beam_ankle_top: axis 0 0 1 -> 0 0 -1; origin xyz=-0.165 0 0 rpy=0 0 0 -> xyz=-0.165 0 0 rpy=3.14159 0 0

Commit message: Sim running multiple robots + controllers. Scripts not updated yet

File: inchworm_description/urdf/inchworm_description.urdf (robot description, URDF)
Before this commit: robot inchworm, 7 links, 6 joints
Links:
- removed link iw_ankle_bottom
- removed link iw_ankle_top
- removed link iw_beam_bottom
- removed link iw_beam_top
- removed link iw_foot_bottom
- removed link iw_foot_top
- removed link iw_root
- added link iw_ankle_bottom_$(arg idx), mass 0.151; collision box size=0.045 0.08 0.08; visual mesh filename=package://inchworm_description/meshes/ankle_bottom.stl scale=0.001 0.001 0.001
- added link iw_ankle_top_$(arg idx), mass 0.151; collision box size=0.08 0.045 0.08; visual mesh filename=package://inchworm_description/meshes/ankle_top.stl scale=0.001 0.001 0.001
- added link iw_beam_bottom_$(arg idx), mass 0.151; collision box size=0.22 0.05 0.08; visual mesh filename=package://inchworm_description/meshes/beam_bottom.stl scale=0.001 0.001 0.001
- added link iw_beam_top_$(arg idx), mass 0.151; collision box size=0.22 0.05 0.08; visual mesh filename=package://inchworm_description/meshes/beam_top.stl scale=0.001 0.001 0.001
- added link iw_foot_bottom_$(arg idx), mass 0.151; collision box size=0.07 0.07 0.05463; visual mesh filename=package://inchworm_description/meshes/ee.stl scale=0.001 0.001 0.001
- added link iw_foot_top_$(arg idx), mass 0.151; collision box size=0.07 0.07 0.05463; visual mesh filename=package://inchworm_description/meshes/ee.stl scale=0.001 0.001 0.001
- added link iw_root_$(arg idx)
Joints:
- removed joint foot_to_root
- removed joint iw_ankle_foot_bottom
- removed joint iw_ankle_foot_top
- removed joint iw_beam_ankle_bottom
- removed joint iw_beam_ankle_top
- removed joint iw_mid_joint
- added joint foot_to_root_$(arg idx): type fixed, parent iw_root_$(arg idx), child iw_foot_bottom_$(arg idx), origin xyz=0 0 0 rpy=0 0 0, limit lower=0 upper=0 effort=10 velocity=10
- added joint iw_ankle_foot_bottom_$(arg idx): type revolute, parent iw_foot_bottom_$(arg idx), child iw_ankle_bottom_$(arg idx), origin xyz=0 0.0075 0.109 rpy=1.57 0 0, axis 0 -1 0, limit lower=-3.14 upper=3.14 effort=10 velocity=1.0
- added joint iw_ankle_foot_top_$(arg idx): type revolute, parent iw_ankle_top_$(arg idx), child iw_foot_top_$(arg idx), origin xyz=-0.109 0 -0.008 rpy=0 1.57 0, axis 0 0 -1, limit lower=-3.14 upper=3.14 effort=10 velocity=1.0
- added joint iw_beam_ankle_bottom_$(arg idx): type revolute, parent iw_ankle_bottom_$(arg idx), child iw_beam_bottom_$(arg idx), origin xyz=0 0 0.0165 rpy=0 0 1.57, axis 0 0 -1, limit lower=-0.785 upper=3.14 effort=10 velocity=1.0
- added joint iw_beam_ankle_top_$(arg idx): type revolute, parent iw_beam_top_$(arg idx), child iw_ankle_top_$(arg idx), origin xyz=-0.165 0 0 rpy=3.14159 0 0, axis 0 0 -1, limit lower=-0.785 upper=3.14 effort=10 velocity=1.0
- added joint iw_mid_joint_$(arg idx): type revolute, parent iw_beam_bottom_$(arg idx), child iw_beam_top_$(arg idx), origin xyz=0.165 0 -0.001 rpy=3.14 0 3.14, axis 0 0 1, limit lower=-0.785 upper=3.14 effort=10 velocity=1.0

Commit message: Old commit from before break, working on hardware testing

File: inchworm_description/urdf/inchworm_description.urdf (robot description, URDF)
Before this commit: robot inchworm, 7 links, 6 joints
Links:
- removed link iw_root
- added link world
Joints:
- joint foot_to_root: parent iw_root -> world
