Commit message: Spawns in a shingle... sort of

File: inchworm_description/urdf/shingle.urdf (robot description, URDF)
Before this commit: robot shingle, 2 links, 0 joints
Links:
- link body: mass None -> 0.151; geometry collision box size=0.013652 0.183003 0.254; collision box size=0.087122 0.014478 0.254
Joints:
- added joint shingle_to_world: type fixed, parent world, child body, origin xyz=0 0 0 rpy=0 0 0

Commit message: fix shingle.urdf to spawn correctly

File: inchworm_description/urdf/shingle.urdf (robot description, URDF)
Before this commit: robot shingle, 2 links, 1 joints
Joints:
- joint shingle_to_world: origin xyz=0 0 0 rpy=0 0 0 -> xyz=0 0 0 rpy=1.57908 0 0

Commit message: Shingles aligned properly

File: inchworm_description/urdf/shingle.urdf (robot description, URDF)
Before this commit: robot shingle, 2 links, 1 joints
Links:
- removed link body
- added link shingle, mass 0.151; collision box size=0.013652 0.183003 0.254; collision box size=0.087122 0.014478 0.254
Joints:
- removed joint shingle_to_world

Commit message: Pick and place now kind of works

File: inchworm_description/urdf/shingle.urdf (robot description, URDF)
Before this commit: robot shingle, 1 links, 0 joints
Links:
- link shingle: mass 0.151 -> 0.0551

Commit message: Shrink shingle collision slightly

File: inchworm_description/urdf/shingle.urdf (robot description, URDF)
Before this commit: robot shingle, 1 links, 0 joints
Links:
- link shingle: geometry collision box size=0.0075 0.17 0.235; collision box size=0.075 0.01 0.235
